Commit message: Restore fingertips after gripper/fingertip xacro split.

File: urdf/diana_gripper_standalone.xacro (robot description, xacro)
@@ -6,5 +6,44 @@
    -->
   <xacro:include filename="$(find diana_gripper)/urdf/diana_gripper.xacro" />
+  <xacro:include filename="$(find diana_gripper)/urdf/fingertips.xacro" />
   <xacro:diana_gripper name="diana_gripper" />
+  <xacro:finray_ridges_fingertip name="diana_gripper/left_finger_finray" />
+  <joint name="diana_gripper/left_finger_finray_joint" type="fixed" >
+    <parent link="diana_gripper/left_finger_tip_mount" />
+    <child  link="diana_gripper/left_finger_finray" />
+    <origin xyz="0.02 0 -0.01" rpy="1.571 0 3.1415" />
+  </joint>
+  <xacro:finray_ridges_fingertip name="diana_gripper/right_finger_finray" />
+  <joint name="diana_gripper/right_finger_finray_joint" type="fixed" >
+    <parent link="diana_gripper/right_finger_tip_mount" />
+    <child  link="diana_gripper/right_finger_finray" />
+    <origin xyz="-0.02 0 -0.01" rpy="1.571 0 0" />
+  </joint>
+  <!-- -->
+  <xacro:digit_fingertip name="diana_gripper/left_finger_digit_sensor" />
+  <xacro:digit_fingertip name="diana_gripper/right_finger_digit_sensor" />
+  <joint name="diana_gripper/left_finger_digit_sensor_joint" type="fixed" >
+    <parent link="diana_gripper/left_finger_tip_mount" />
+    <child  link="diana_gripper/left_finger_digit_sensor" />
+    <origin xyz="0 0 0" rpy="0 0 -1.571" />
+  </joint>
+  <joint name="diana_gripper/right_finger_digit_sensor_joint" type="fixed" >
+    <parent link="diana_gripper/right_finger_tip_mount" />
+    <child  link="diana_gripper/right_finger_digit_sensor" />
+    <origin xyz="0 0 0" rpy="0 0 1.571" />
+  </joint>
+  <!-- -->
+  <xacro:simple_fingertip name="diana_gripper/left_finger_simple_fingertip" />
+  <xacro:simple_fingertip name="diana_gripper/right_finger_simple_fingertip" />
+  <joint name="diana_gripper/left_fingertip_simple_joint" type="fixed" >
+    <parent link="diana_gripper/left_finger_tip_mount" />
+    <child  link="diana_gripper/left_finger_simple_fingertip" />
+    <origin xyz="0 0 0" rpy="0 0 1.571" />
+  </joint>
+  <joint name="diana_gripper/right_fingertip_simple_joint" type="fixed" >
+    <parent link="diana_gripper/right_finger_tip_mount" />
+    <child  link="diana_gripper/right_finger_simple_fingertip" />
+    <origin xyz="0 0 0" rpy="0 0 -1.571" />
+  </joint>
   <link name="world" />
   <joint name="world_diana_gripper_joint" type="fixed" >

Commit message: Demo gripper with one DIGIT sensor and one simple fingertip.

File: urdf/diana_gripper_standalone.xacro (robot description, xacro)
@@ -7,10 +7,19 @@
   <xacro:include filename="$(find diana_gripper)/urdf/diana_gripper.xacro" />
   <xacro:include filename="$(find diana_gripper)/urdf/fingertips.xacro" />
+  <!-- the world frame -->
+  <link name="world" />
+  <!-- the gripper, attached to world -->
   <xacro:diana_gripper name="diana_gripper" />
+  <joint name="world_diana_gripper_joint" type="fixed" >
+   <parent link="world" />
+   <child  link="diana_gripper" />
+   <origin xyz="0 0 0.1" rpy="0 0 0" />
+  </joint>
+  <!-- uncomment to use finray fingertips:
   <xacro:finray_ridges_fingertip name="diana_gripper/left_finger_finray" />
   <joint name="diana_gripper/left_finger_finray_joint" type="fixed" >
     <parent link="diana_gripper/left_finger_tip_mount" />
     <child  link="diana_gripper/left_finger_finray" />
-    <origin xyz="0.02 0 -0.01" rpy="1.571 0 3.1415" />
+    <origin xyz="0 0 0" rpy="1.571 0 3.1415" />
   </joint>
   <xacro:finray_ridges_fingertip name="diana_gripper/right_finger_finray" />
@@ -18,9 +27,9 @@
     <parent link="diana_gripper/right_finger_tip_mount" />
     <child  link="diana_gripper/right_finger_finray" />
-    <origin xyz="-0.02 0 -0.01" rpy="1.571 0 0" />
+    <origin xyz="0 0 0" rpy="1.571 0 0" />
   </joint>
-  <!-- -->
+  -->
+  <!-- uncomment to use left-finger digit sensor:
   <xacro:digit_fingertip name="diana_gripper/left_finger_digit_sensor" />
-  <xacro:digit_fingertip name="diana_gripper/right_finger_digit_sensor" />
   <joint name="diana_gripper/left_finger_digit_sensor_joint" type="fixed" >
     <parent link="diana_gripper/left_finger_tip_mount" />
@@ -28,4 +37,7 @@
     <origin xyz="0 0 0" rpy="0 0 -1.571" />
   </joint>
+  -->
+  <!-- a digit sensor on the right finger -->
+  <xacro:digit_fingertip name="diana_gripper/right_finger_digit_sensor" />
   <joint name="diana_gripper/right_finger_digit_sensor_joint" type="fixed" >
     <parent link="diana_gripper/right_finger_tip_mount" />
@@ -33,7 +45,6 @@
     <origin xyz="0 0 0" rpy="0 0 1.571" />
   </joint>
-  <!-- -->
+  <!-- a simple (pyramid shape) fingertip on the left finger -->
   <xacro:simple_fingertip name="diana_gripper/left_finger_simple_fingertip" />
-  <xacro:simple_fingertip name="diana_gripper/right_finger_simple_fingertip" />
   <joint name="diana_gripper/left_fingertip_simple_joint" type="fixed" >
     <parent link="diana_gripper/left_finger_tip_mount" />
@@ -41,4 +52,6 @@
     <origin xyz="0 0 0" rpy="0 0 1.571" />
   </joint>
+  <!-- uncomment for the simple (pyramid) fingertip on the right finger:
+  <xacro:simple_fingertip name="diana_gripper/right_finger_simple_fingertip" />
   <joint name="diana_gripper/right_fingertip_simple_joint" type="fixed" >
     <parent link="diana_gripper/right_finger_tip_mount" />
@@ -46,9 +59,4 @@
     <origin xyz="0 0 0" rpy="0 0 -1.571" />
   </joint>
-  <link name="world" />
-  <joint name="world_diana_gripper_joint" type="fixed" >
-   <parent link="world" />
-   <child  link="diana_gripper" />
-   <origin xyz="0 0 0.1" rpy="0 0 0" />
-  </joint>
+  -->
 </robot>
