Commit message: Larger proximal tilt joint range for dual-use DIGIT gripper.

File: urdf/fake_parallel_gripper.xacro (robot description, xacro)
@@ -40,5 +40,6 @@
     <origin xyz="0 0 0" rpy="0 0 0" />
     <axis xyz="0 0 1" />
-    <limit lower="-1.2" upper="1.2" effort="1" velocity="1" />
+    <!-- extra large joint limit 2.0 for "combined" DigitSensor gripper, use 1.57 otherwise -->
+    <limit lower="-2.0" upper="2.0" effort="1" velocity="1" />
   </joint>
   <link name="world" />
