Commit message: integrated multitip fingertip

File: urdf/fingertips.xacro (robot description, xacro)
@@ -1,6 +1,6 @@
 <?xml version="1.0" ?>
 <robot xmlns:xacro="http://www.ros.org/wiki/xacro" name="digit_fingertip">
- <xacro:macro name="digit_fingertip" params="name">
-  <!-- digit sensors on the distal finger brackets -->
+<xacro:macro name="digit_fingertip" params="name">
+<!-- digit sensors on the distal finger brackets -->
   <link name="${name}" >
     <visual>
@@ -17,4 +17,24 @@
       <geometry>
         <mesh filename="package://diana_gripper/meshes/digit_sensor.stl" scale="0.001 0.001 0.001" />
+      </geometry>
+    </collision>
+  </link>
+</xacro:macro>
+<xacro:macro name="digit_multitip_fingertip" params="name">
+<!-- digit sensors on the distal finger brackets -->
+  <link name="${name}" >
+    <visual>
+      <origin xyz="0 -0.01 0" rpy="0 0 3.141" />
+      <material name="${name}_material" >
+        <color rgba="0.4 0.4 0.4 1.0" />
+      </material>
+      <geometry>
+        <mesh filename="package://diana_gripper/meshes/multitip.stl" scale="0.001 0.001 0.001" />
+      </geometry>
+    </visual>
+    <collision>
+      <origin xyz="0 -0.01 0" rpy="0 0 3.141" />
+      <geometry>
+        <mesh filename="package://diana_gripper/meshes/multitip_hull.stl" scale="0.001 0.001 0.001" />
       </geometry>
     </collision>

Commit message: Add (fake) inertial blocks for Gazebo simulation.

File: urdf/fingertips.xacro (robot description, xacro)
@@ -4,4 +4,9 @@
 <!-- digit sensors on the distal finger brackets -->
   <link name="${name}" >
+    <inertial>
+      <origin xyz="0 0 0" rpy="0 0 0"/>
+      <mass value="0.051" />
+      <inertia ixx="0.001" ixy="0" ixz="0" iyy="0.001" iyz="0" izz="0.001" />
+    </inertial>
     <visual>
       <origin xyz="0 0 0" rpy="0 0 1.571" />
@@ -24,4 +29,9 @@
 <!-- digit sensors on the distal finger brackets -->
   <link name="${name}" >
+    <inertial>
+      <origin xyz="0 0 0" rpy="0 0 0"/>
+      <mass value="0.051" />
+      <inertia ixx="0.001" ixy="0" ixz="0" iyy="0.001" iyz="0" izz="0.001" />
+    </inertial>
     <visual>
       <origin xyz="0 -0.01 0" rpy="0 0 3.141" />
@@ -44,4 +54,9 @@
   <!-- simple finger brackets -->
   <link name="${name}" >
+    <inertial>
+      <origin xyz="0 0 0" rpy="0 0 0"/>
+      <mass value="0.011" />
+      <inertia ixx="0.001" ixy="0" ixz="0" iyy="0.001" iyz="0" izz="0.001" />
+    </inertial>
     <visual>
       <origin xyz="0 0 0" rpy="0 0 0" />
@@ -63,4 +78,9 @@
 <xacro:macro name="finray_fingertip" params="name">
   <link name="${name}" >
+    <inertial>
+      <origin xyz="0 0 0" rpy="0 0 0"/>
+      <mass value="0.021" />
+      <inertia ixx="0.001" ixy="0" ixz="0" iyy="0.001" iyz="0" izz="0.001" />
+    </inertial>
     <visual>
       <origin xyz="0 0 0" rpy="0 0 0" />
@@ -76,4 +96,9 @@
 <xacro:macro name="finray_ridges_fingertip" params="name">
   <link name="${name}" >
+    <inertial>
+      <origin xyz="0 0 0" rpy="0 0 0"/>
+      <mass value="0.021" />
+      <inertia ixx="0.001" ixy="0" ixz="0" iyy="0.001" iyz="0" izz="0.001" />
+    </inertial>
     <visual>
       <origin xyz="0 0 0" rpy="0 0 0" />
