Commit message: Rename fingertip-mount frames; separate fingertips.

File: urdf/diana_gripper.xacro (robot description, xacro)
@@ -2,7 +2,8 @@
 <robot xmlns:xacro="http://www.ros.org/wiki/xacro" name="diana_gripper">
   <xacro:property name="KG_CM" value="1" />   <!-- actually: 0.0981 to convert from kg*cm to N*m -->
-  <xacro:include filename="$(find scservo)/urdf/scservo.xacro" />
+  <xacro:include filename="$(find diana_gripper)/urdf/scservo.xacro" />
   <xacro:include filename="$(find diana_gripper)/urdf/diana_gripper_gazebo.xacro" />
-  <xacro:include filename="$(find scservo)/urdf/fingertip.xacro" />
+  <xacro:include filename="$(find diana_gripper)/urdf/imu_gy521.xacro" />
+  <xacro:include filename="$(find diana_gripper)/urdf/fingertip.xacro" />
   <xacro:diana_gripper_control_plugin name="diana_gripper" />
 <xacro:macro name="diana_gripper" params="name" >
@@ -132,10 +133,9 @@
     </actuator>
   </transmission>
-  <xacro:fingertip name="diana_gripper/left_finger_fingertip" radius="0.010"
-                      rgba="1.0 0.0 0.0 1.0" gmaterial="Gazebo/Red" />
+  <link name="diana_gripper/left_finger_tip_mount" />
   <!-- convert from weird SCS20 coordinates back to base frame (when finger straight) -->
-  <joint name="diana_gripper/left_finger_fingertip_joint" type="fixed">
+  <joint name="diana_gripper/left_finger_tip_mount_joint" type="fixed">
     <parent link="diana_gripper/left_finger_distal_bracket" />
-    <child  link="diana_gripper/left_finger_fingertip" />
+    <child  link="diana_gripper/left_finger_tip_mount" />
     <origin xyz="0 0 ${-0.0275}" rpy="0 3.1415 0" />
   </joint>
@@ -211,14 +211,37 @@
     </actuator>
   </transmission>
-  <xacro:fingertip name="diana_gripper/right_finger_fingertip" radius="0.010"
-                      rgba="0.0 1.0 0.0 1.0" gmaterial="Gazebo/Green" />
+  <link name="diana_gripper/right_finger_tip_mount" />
   <!-- convert from weird SCS20 coordinates back to base frame (when finger straight) -->
-  <joint name="diana_gripper/right_finger_fingertip_joint" type="fixed">
+  <joint name="diana_gripper/right_finger_tip_mount_joint" type="fixed">
     <parent link="diana_gripper/right_finger_distal_bracket" />
-    <child  link="diana_gripper/right_finger_fingertip" />
+    <child  link="diana_gripper/right_finger_tip_mount" />
     <origin xyz="0 0 ${-0.0275}" rpy="0 3.1415 0" />   <!-- or ${-0.0275-0.02} -->
   </joint>
+  <xacro:dummy_fingertips/>
   <xacro:digit_fingertips/>
   <xacro:finray_fingertips/>
+  <!-- <xacro:finray_ridges_fingertips/> -->
+  <xacro:imu_gy521 parent="diana_gripper/left_finger_tip_mount" name="diana_gripper/left_finger_imu" >
+    <origin xyz="0 0.023 0" rpy="0 0 3.141" />
+  </xacro:imu_gy521>
+  <xacro:imu_gy521 parent="diana_gripper/right_finger_tip_mount" name="diana_gripper/right_finger_imu" >
+    <origin xyz="0 0.023 0" rpy="0 0 3.141" />
+  </xacro:imu_gy521>
+</xacro:macro> <!-- end xacro:diana_gripper -->
+<xacro:macro name="dummy_fingertips" >
+  <xacro:fingertip name="diana_gripper/left_finger_fingertip" radius="0.005"
+                      rgba="1.0 0.0 0.0 1.0" gmaterial="Gazebo/Red" />
+  <joint name="diana_gripper/left_finger_fingertip_joint" type="fixed">
+    <parent link="diana_gripper/left_finger_tip_mount" />
+    <child  link="diana_gripper/left_finger_fingertip" />
+    <origin xyz="+0.02 0 0.07" rpy="0 0 0" />
+  </joint>
+  <xacro:fingertip name="diana_gripper/right_finger_fingertip" radius="0.005"
+                      rgba="0.0 1.0 0.0 1.0" gmaterial="Gazebo/Green" />
+  <joint name="diana_gripper/right_finger_fingertip_joint" type="fixed">
+    <parent link="diana_gripper/right_finger_tip_mount" />
+    <child  link="diana_gripper/right_finger_fingertip" />
+    <origin xyz="-0.02 0 0.07" rpy="0 0 0" />
+  </joint>
 </xacro:macro>
 <xacro:macro name="digit_fingertips" >
@@ -236,5 +259,5 @@
   </link>
   <joint name="diana_gripper/left_finger_digit_sensor_joint" type="fixed" >
-    <parent link="diana_gripper/left_finger_fingertip" />
+    <parent link="diana_gripper/left_finger_tip_mount" />
     <child  link="diana_gripper/left_finger_digit_sensor" />
     <origin xyz="0 0 0" rpy="0 0 -1.571" />
@@ -252,5 +275,5 @@
   </link>
   <joint name="diana_gripper/right_finger_digit_sensor_joint" type="fixed" >
-    <parent link="diana_gripper/right_finger_fingertip" />
+    <parent link="diana_gripper/right_finger_tip_mount" />
     <child  link="diana_gripper/right_finger_digit_sensor" />
     <origin xyz="0 0 0" rpy="0 0 1.571" />
@@ -270,5 +293,5 @@
   </link>
   <joint name="diana_gripper/left_finger_finray_joint" type="fixed" >
-    <parent link="diana_gripper/left_finger_fingertip" />
+    <parent link="diana_gripper/left_finger_tip_mount" />
     <child  link="diana_gripper/left_finger_finray" />
     <origin xyz="0.02 0 -0.01" rpy="1.571 0 3.1415" />
@@ -286,7 +309,41 @@
   </link>
   <joint name="diana_gripper/right_finger_finray_joint" type="fixed" >
-    <parent link="diana_gripper/right_finger_fingertip" />
+    <parent link="diana_gripper/right_finger_tip_mount" />
     <child  link="diana_gripper/right_finger_finray" />
     <origin xyz="-0.02 0 -0.01" rpy="1.571 0 0" />
+  </joint>
+</xacro:macro>
+<xacro:macro name="finray_ridges_fingertips">
+  <link name="diana_gripper/left_finger_finray_ridges" >
+    <visual>
+      <origin xyz="0 0 0" rpy="0 0 0" />
+      <material name="diana_gripper_left_finger_finray_ridges_material" >
+        <color rgba="0.4 0.4 0.4 1.0" />
+      </material>
+      <geometry>
+        <mesh filename="package://diana_gripper/meshes/finray_finger_slanted_ridges.stl" scale="0.001 0.001 0.001" />
+      </geometry>
+    </visual>
+  </link>
+  <joint name="diana_gripper/left_finger_finray_ridges_joint" type="fixed" >
+    <parent link="diana_gripper/left_finger_tip_mount" />
+    <child  link="diana_gripper/left_finger_finray_ridges" />
+    <origin xyz="0 0 0" rpy="1.571 0 3.1415" />
+  </joint>
+  <link name="diana_gripper/right_finger_finray_ridges" >
+    <visual>
+      <origin xyz="0 0 0" rpy="0 0 0" />
+      <material name="diana_gripper_right_finger_finray_ridges_material" >
+        <color rgba="0.4 0.4 0.4 1.0" />
+      </material>
+      <geometry>
+        <mesh filename="package://diana_gripper/meshes/finray_finger_slanted_ridges.stl" scale="0.001 0.001 0.001" />
+      </geometry>
+    </visual>
+  </link>
+  <joint name="diana_gripper/right_finger_finray_ridges_joint" type="fixed" >
+    <parent link="diana_gripper/right_finger_tip_mount" />
+    <child  link="diana_gripper/right_finger_finray_ridges" />
+    <origin xyz="0 0 0" rpy="1.571 0 0" />
   </joint>
 </xacro:macro>

Commit message: add simple_fingertips to urdf

File: urdf/diana_gripper.xacro (robot description, xacro)
@@ -218,8 +218,9 @@
     <origin xyz="0 0 ${-0.0275}" rpy="0 3.1415 0" />   <!-- or ${-0.0275-0.02} -->
   </joint>
-  <xacro:dummy_fingertips/>
+  <!-- <xacro:dummy_fingertips/>
   <xacro:digit_fingertips/>
   <xacro:finray_fingertips/>
-  <!-- <xacro:finray_ridges_fingertips/> -->
+  <xacro:finray_ridges_fingertips/> -->
+  <xacro:simple_fingertips/>
   <xacro:imu_gy521 parent="diana_gripper/left_finger_tip_mount" name="diana_gripper/left_finger_imu" >
     <origin xyz="0 0.023 0" rpy="0 0 3.141" />
@@ -280,4 +281,39 @@
   </joint>
 </xacro:macro>
+<xacro:macro name="simple_fingertips" >
+  <!-- simple finger brackets -->
+  <link name="diana_gripper/left_fingertip_simple" >
+    <visual>
+      <origin xyz="0 0 0" rpy="0 0 0" />
+      <material name="diana_gripper_left_fingertip_simple_material" >
+        <color rgba="0.95 1 0 1.0" />
+      </material>
+      <geometry>
+        <mesh filename="package://diana_gripper/meshes/fingertip_simple.stl" scale="0.001 0.001 0.001" />
+      </geometry>
+    </visual>
+  </link>
+  <joint name="diana_gripper/left_fingertip_simple_joint" type="fixed" >
+    <parent link="diana_gripper/left_finger_tip_mount" />
+    <child  link="diana_gripper/left_fingertip_simple" />
+    <origin xyz="0 0 0" rpy="0 0 1.571" />
+  </joint>
+  <link name="diana_gripper/right_fingertip_simple" >
+    <visual>
+      <origin xyz="0 0 0" rpy="0 0 0" />
+      <material name="diana_gripper_right_fingertip_simple_material" >
+        <color rgba="0.95 1 0 1.0" />
+      </material>
+      <geometry>
+        <mesh filename="package://diana_gripper/meshes/fingertip_simple.stl" scale="0.001 0.001 0.001" />
+      </geometry>
+    </visual>
+  </link>
+  <joint name="diana_gripper/right_fingertip_simple_joint" type="fixed" >
+    <parent link="diana_gripper/right_finger_tip_mount" />
+    <child  link="diana_gripper/right_fingertip_simple" />
+    <origin xyz="0 0 0" rpy="0 0 -1.571" />
+  </joint>
+</xacro:macro>
 <xacro:macro name="finray_fingertips">
   <link name="diana_gripper/left_finger_finray" >

Commit message: add tcp to urdf

File: urdf/diana_gripper.xacro (robot description, xacro)
@@ -223,4 +223,5 @@
   <xacro:finray_ridges_fingertips/> -->
   <xacro:simple_fingertips/>
+  <xacro:tcp/>
   <xacro:imu_gy521 parent="diana_gripper/left_finger_tip_mount" name="diana_gripper/left_finger_imu" >
     <origin xyz="0 0.023 0" rpy="0 0 3.141" />
@@ -384,4 +385,16 @@
   </joint>
 </xacro:macro>
+<xacro:macro name="tcp">
+  <link name="diana_gripper/tcp" >
+    <visual>
+      <origin xyz="0 0 0" rpy="0 0 0" />
+    </visual>
+  </link>
+  <joint name="diana_gripper/tcp_joint" type="fixed" >
+    <parent link="diana_gripper" />
+    <child  link="diana_gripper/tcp" />
+    <origin xyz="0 0 0.15" rpy="0 0 0" />
+  </joint>
+</xacro:macro>
 <!--
   <link name="world" />

Commit message: added more collision geometries to urdf

File: urdf/diana_gripper.xacro (robot description, xacro)
@@ -32,5 +32,5 @@
         <origin xyz="0 0 ${(0.02+0.0127)/2}" rpy="0 0 0" />
         <geometry>
-          <box size="${0.075*2} 0.085 ${0.02+0.0127}" />
+          <box size="${0.075*2} 0.105 ${0.02+0.0127}" />
         </geometry>
       </collision>
@@ -97,4 +97,10 @@
       </geometry>
     </visual>
+    <collision>
+      <origin xyz="0 0.001 0" rpy="0 -1.571 0" />
+      <geometry>
+        <mesh filename="package://diana_gripper/meshes/diana_gripper_connector_v1.stl" scale="0.001 0.001 0.001" />
+      </geometry>
+    </collision>
   </link>
   <joint name="diana_gripper/left_finger_distal_servo_mount_joint" type="fixed" >
@@ -113,4 +119,10 @@
       </geometry>
     </visual>
+    <collision>
+      <origin xyz="0 0 -0.0275" rpy="0 0 1.571" />
+      <geometry>
+        <mesh filename="package://diana_gripper/meshes/feetech_bracket_big.stl" scale="0.001 0.001 0.001" />
+      </geometry>
+    </collision>
   </link>
   <joint name="diana_gripper/LFJ1" type="revolute" >
@@ -175,4 +187,10 @@
       </geometry>
     </visual>
+    <collision>
+      <origin xyz="0 0.001 0" rpy="0 -1.571 0" />
+      <geometry>
+        <mesh filename="package://diana_gripper/meshes/diana_gripper_connector_v1.stl" scale="0.001 0.001 0.001" />
+      </geometry>
+    </collision>
   </link>
   <joint name="diana_gripper/right_finger_distal_servo_mount_joint" type="fixed" >
@@ -191,4 +209,10 @@
       </geometry>
     </visual>
+    <collision>
+      <origin xyz="0 0 -0.0275" rpy="0 0 1.571" />
+      <geometry>
+        <mesh filename="package://diana_gripper/meshes/feetech_bracket_big.stl" scale="0.001 0.001 0.001" />
+      </geometry>
+    </collision>
   </link>
   <joint name="diana_gripper/RFJ1" type="revolute" >
@@ -259,4 +283,10 @@
       </geometry>
     </visual>
+    <collision>
+      <origin xyz="0 0 0" rpy="0 0 1.571" />
+      <geometry>
+        <mesh filename="package://diana_gripper/meshes/digit_sensor.stl" scale="0.001 0.001 0.001" />
+      </geometry>
+    </collision>
   </link>
   <joint name="diana_gripper/left_finger_digit_sensor_joint" type="fixed" >
@@ -275,4 +305,10 @@
       </geometry>
     </visual>
+    <collision>
+      <origin xyz="0 0 0" rpy="0 0 1.571" />
+      <geometry>
+        <mesh filename="package://diana_gripper/meshes/digit_sensor.stl" scale="0.001 0.001 0.001" />
+      </geometry>
+    </collision>
   </link>
   <joint name="diana_gripper/right_finger_digit_sensor_joint" type="fixed" >
@@ -294,4 +330,10 @@
       </geometry>
     </visual>
+    <collision>
+      <origin xyz="0 0 0" rpy="0 0 0" />
+      <geometry>
+        <mesh filename="package://diana_gripper/meshes/fingertip_simple_hull.stl" scale="0.001 0.001 0.001" />
+      </geometry>
+    </collision>
   </link>
   <joint name="diana_gripper/left_fingertip_simple_joint" type="fixed" >
@@ -310,4 +352,10 @@
       </geometry>
     </visual>
+    <collision>
+      <origin xyz="0 0 0" rpy="0 0 0" />
+      <geometry>
+        <mesh filename="package://diana_gripper/meshes/fingertip_simple_hull.stl" scale="0.001 0.001 0.001" />
+      </geometry>
+    </collision>
   </link>
   <joint name="diana_gripper/right_fingertip_simple_joint" type="fixed" >

Commit message: increased gripper joint velocity limits

File: urdf/diana_gripper.xacro (robot description, xacro)
@@ -73,5 +73,5 @@
     <origin xyz="0 0 0" rpy="0 0 0" />
     <axis xyz="0 1 0" />
-    <limit lower="-1.571" upper="+1.571" effort="1" velocity="0.5" />
+    <limit lower="-1.571" upper="+1.571" effort="1" velocity="6.28" />
     <dynamics damping="0.7" friction="0.0" />
     <safety_controller soft_lower_limit="-1.57" soft_upper_limit="1.57" k_position="1000" k_velocity="100"/>
@@ -131,5 +131,5 @@
     <origin xyz="0 0 0" rpy="0 0 0" />
     <axis xyz="0 1 0" />
-    <limit lower="-2.21" upper="+2.21" effort="1" velocity="0.5" />
+    <limit lower="-2.21" upper="+2.21" effort="1" velocity="6.28" />
     <dynamics damping="0.7" friction="0.0" />
     <safety_controller soft_lower_limit="-2.20" soft_upper_limit="2.20" k_position="1000" k_velocity="100"/>
@@ -163,5 +163,5 @@
     <origin xyz="0 0 0" rpy="0 0 0" />
     <axis xyz="0 -1 0" />
-    <limit lower="-1.571" upper="+1.571" effort="1" velocity="0.5" />
+    <limit lower="-1.571" upper="+1.571" effort="1" velocity="6.28" />
     <dynamics damping="0.7" friction="0.0" />
     <safety_controller soft_lower_limit="-1.57" soft_upper_limit="1.57" k_position="1000" k_velocity="100"/>
@@ -221,5 +221,5 @@
     <origin xyz="0 0 0" rpy="0 0 0" />
     <axis xyz="0 -1 0" />
-    <limit lower="-2.21" upper="+2.21" effort="1" velocity="0.5" />
+    <limit lower="-2.21" upper="+2.21" effort="1" velocity="6.28" />
     <dynamics damping="0.7" friction="0.0" />
     <safety_controller soft_lower_limit="-2.20" soft_upper_limit="2.20" k_position="1000" k_velocity="100"/>

Commit message: fixed tcp link

File: urdf/diana_gripper.xacro (robot description, xacro)
@@ -435,7 +435,4 @@
 <xacro:macro name="tcp">
   <link name="diana_gripper/tcp" >
-    <visual>
-      <origin xyz="0 0 0" rpy="0 0 0" />
-    </visual>
   </link>
   <joint name="diana_gripper/tcp_joint" type="fixed" >

Commit message: move fingertips into separate file

File: urdf/diana_gripper.xacro (robot description, xacro)
@@ -245,6 +245,6 @@
   <xacro:digit_fingertips/>
   <xacro:finray_fingertips/>
-  <xacro:finray_ridges_fingertips/> -->
-  <xacro:simple_fingertips/>
+  <xacro:finray_ridges_fingertips/>
+  <xacro:simple_fingertips/>  -->
   <xacro:tcp/>
   <xacro:imu_gy521 parent="diana_gripper/left_finger_tip_mount" name="diana_gripper/left_finger_imu" >
@@ -271,166 +271,4 @@
   </joint>
 </xacro:macro>
-<xacro:macro name="digit_fingertips" >
-  <!-- digit sensors on the distal finger brackets -->
-  <link name="diana_gripper/left_finger_digit_sensor" >
-    <visual>
-      <origin xyz="0 0 0" rpy="0 0 1.571" />
-      <material name="diana_gripper_left_finger_distal_sensor_material" >
-        <color rgba="0.4 0.4 0.4 1.0" />
-      </material>
-      <geometry>
-        <mesh filename="package://diana_gripper/meshes/digit_sensor.stl" scale="0.001 0.001 0.001" />
-      </geometry>
-    </visual>
-    <collision>
-      <origin xyz="0 0 0" rpy="0 0 1.571" />
-      <geometry>
-        <mesh filename="package://diana_gripper/meshes/digit_sensor.stl" scale="0.001 0.001 0.001" />
-      </geometry>
-    </collision>
-  </link>
-  <joint name="diana_gripper/left_finger_digit_sensor_joint" type="fixed" >
-    <parent link="diana_gripper/left_finger_tip_mount" />
-    <child  link="diana_gripper/left_finger_digit_sensor" />
-    <origin xyz="0 0 0" rpy="0 0 -1.571" />
-  </joint>
-  <link name="diana_gripper/right_finger_digit_sensor" >
-    <visual>
-      <origin xyz="0 0 0" rpy="0 0 1.571" />
-      <material name="diana_gripper_right_finger_distal_sensor_material" >
-        <color rgba="0.4 0.4 0.4 1.0" />
-      </material>
-      <geometry>
-        <mesh filename="package://diana_gripper/meshes/digit_sensor.stl" scale="0.001 0.001 0.001" />
-      </geometry>
-    </visual>
-    <collision>
-      <origin xyz="0 0 0" rpy="0 0 1.571" />
-      <geometry>
-        <mesh filename="package://diana_gripper/meshes/digit_sensor.stl" scale="0.001 0.001 0.001" />
-      </geometry>
-    </collision>
-  </link>
-  <joint name="diana_gripper/right_finger_digit_sensor_joint" type="fixed" >
-    <parent link="diana_gripper/right_finger_tip_mount" />
-    <child  link="diana_gripper/right_finger_digit_sensor" />
-    <origin xyz="0 0 0" rpy="0 0 1.571" />
-  </joint>
-</xacro:macro>
-<xacro:macro name="simple_fingertips" >
-  <!-- simple finger brackets -->
-  <link name="diana_gripper/left_fingertip_simple" >
-    <visual>
-      <origin xyz="0 0 0" rpy="0 0 0" />
-      <material name="diana_gripper_left_fingertip_simple_material" >
-        <color rgba="0.95 1 0 1.0" />
-      </material>
-      <geometry>
-        <mesh filename="package://diana_gripper/meshes/fingertip_simple.stl" scale="0.001 0.001 0.001" />
-      </geometry>
-    </visual>
-    <collision>
-      <origin xyz="0 0 0" rpy="0 0 0" />
-      <geometry>
-        <mesh filename="package://diana_gripper/meshes/fingertip_simple_hull.stl" scale="0.001 0.001 0.001" />
-      </geometry>
-    </collision>
-  </link>
-  <joint name="diana_gripper/left_fingertip_simple_joint" type="fixed" >
-    <parent link="diana_gripper/left_finger_tip_mount" />
-    <child  link="diana_gripper/left_fingertip_simple" />
-    <origin xyz="0 0 0" rpy="0 0 1.571" />
-  </joint>
-  <link name="diana_gripper/right_fingertip_simple" >
-    <visual>
-      <origin xyz="0 0 0" rpy="0 0 0" />
-      <material name="diana_gripper_right_fingertip_simple_material" >
-        <color rgba="0.95 1 0 1.0" />
-      </material>
-      <geometry>
-        <mesh filename="package://diana_gripper/meshes/fingertip_simple.stl" scale="0.001 0.001 0.001" />
-      </geometry>
-    </visual>
-    <collision>
-      <origin xyz="0 0 0" rpy="0 0 0" />
-      <geometry>
-        <mesh filename="package://diana_gripper/meshes/fingertip_simple_hull.stl" scale="0.001 0.001 0.001" />
-      </geometry>
-    </collision>
-  </link>
-  <joint name="diana_gripper/right_fingertip_simple_joint" type="fixed" >
-    <parent link="diana_gripper/right_finger_tip_mount" />
-    <child  link="diana_gripper/right_fingertip_simple" />
-    <origin xyz="0 0 0" rpy="0 0 -1.571" />
-  </joint>
-</xacro:macro>
-<xacro:macro name="finray_fingertips">
-  <link name="diana_gripper/left_finger_finray" >
-    <visual>
-      <origin xyz="0 0 0" rpy="0 0 0" />
-      <material name="diana_gripper_left_finger_finray_material" >
-        <color rgba="0.4 0.4 0.4 1.0" />
-      </material>
-      <geometry>
-        <mesh filename="package://diana_gripper/meshes/finray_finger.stl" scale="0.001 0.001 0.001" />
-      </geometry>
-    </visual>
-  </link>
-  <joint name="diana_gripper/left_finger_finray_joint" type="fixed" >
-    <parent link="diana_gripper/left_finger_tip_mount" />
-    <child  link="diana_gripper/left_finger_finray" />
-    <origin xyz="0.02 0 -0.01" rpy="1.571 0 3.1415" />
-  </joint>
-  <link name="diana_gripper/right_finger_finray" >
-    <visual>
-      <origin xyz="0 0 0" rpy="0 0 0" />
-      <material name="diana_gripper_right_finger_finray_material" >
-        <color rgba="0.4 0.4 0.4 1.0" />
-      </material>
-      <geometry>
-        <mesh filename="package://diana_gripper/meshes/finray_finger.stl" scale="0.001 0.001 0.001" />
-      </geometry>
-    </visual>
-  </link>
-  <joint name="diana_gripper/right_finger_finray_joint" type="fixed" >
-    <parent link="diana_gripper/right_finger_tip_mount" />
-    <child  link="diana_gripper/right_finger_finray" />
-    <origin xyz="-0.02 0 -0.01" rpy="1.571 0 0" />
-  </joint>
-</xacro:macro>
-<xacro:macro name="finray_ridges_fingertips">
-  <link name="diana_gripper/left_finger_finray_ridges" >
-    <visual>
-      <origin xyz="0 0 0" rpy="0 0 0" />
-      <material name="diana_gripper_left_finger_finray_ridges_material" >
-        <color rgba="0.4 0.4 0.4 1.0" />
-      </material>
-      <geometry>
-        <mesh filename="package://diana_gripper/meshes/finray_finger_slanted_ridges.stl" scale="0.001 0.001 0.001" />
-      </geometry>
-    </visual>
-  </link>
-  <joint name="diana_gripper/left_finger_finray_ridges_joint" type="fixed" >
-    <parent link="diana_gripper/left_finger_tip_mount" />
-    <child  link="diana_gripper/left_finger_finray_ridges" />
-    <origin xyz="0 0 0" rpy="1.571 0 3.1415" />
-  </joint>
-  <link name="diana_gripper/right_finger_finray_ridges" >
-    <visual>
-      <origin xyz="0 0 0" rpy="0 0 0" />
-      <material name="diana_gripper_right_finger_finray_ridges_material" >
-        <color rgba="0.4 0.4 0.4 1.0" />
-      </material>
-      <geometry>
-        <mesh filename="package://diana_gripper/meshes/finray_finger_slanted_ridges.stl" scale="0.001 0.001 0.001" />
-      </geometry>
-    </visual>
-  </link>
-  <joint name="diana_gripper/right_finger_finray_ridges_joint" type="fixed" >
-    <parent link="diana_gripper/right_finger_tip_mount" />
-    <child  link="diana_gripper/right_finger_finray_ridges" />
-    <origin xyz="0 0 0" rpy="1.571 0 0" />
-  </joint>
-</xacro:macro>
 <xacro:macro name="tcp">
   <link name="diana_gripper/tcp" >
