Commit message: use name parameter in xacro for digit gripper

File: urdf/diana_gripper.xacro (robot description, xacro)
@@ -11,5 +11,5 @@
        Origin is at the bottom center of the base plate.
    -->
-  <link name="diana_gripper">
+  <link name="${name}">
       <inertial>
         <!-- note that estimated mass does not include servos, these are separate -->
@@ -21,5 +21,5 @@
       <visual>
         <origin xyz="0 0 0" />
-        <material name="diana_gripper_base_v1_material" >
+        <material name="${name}_base_v1_material" >
           <color rgba="0.4 0.4 0.4 1.0" />
         </material>
@@ -36,5 +36,5 @@
       </collision>
   </link>
-  <gazebo reference="diana_gripper">
+  <gazebo reference="${name}">
       <material>Gazebo/Black</material>
       <turnGravityOff>false</turnGravityOff>
@@ -47,28 +47,28 @@
   </gazebo>
   <!-- four servos -->
-  <xacro:scservo name="diana_gripper/left_finger_proximal_servo"
-                 type="scs20"
-                 rgba="0.0 0.0 0.6 1.0" gmaterial="Gazebo/Blue">
-  </xacro:scservo>
-  <xacro:scservo name="diana_gripper/left_finger_distal_servo"
-                 type="scs20"
-                 rgba="0.0 0.0 0.6 1.0" gmaterial="Gazebo/Blue">
-  </xacro:scservo>
-  <xacro:scservo name="diana_gripper/right_finger_proximal_servo"
-                 type="scs20"
-                 rgba="0.0 0.0 0.6 1.0" gmaterial="Gazebo/Blue">
-  </xacro:scservo>
-  <xacro:scservo name="diana_gripper/right_finger_distal_servo"
-                 type="scs20"
-                 rgba="0.0 0.0 0.6 1.0" gmaterial="Gazebo/Blue">
-  </xacro:scservo>
-  <joint name="diana_gripper/left_finger_proximal_servo_mount_joint" type="fixed" >
-    <parent link="diana_gripper" />
-    <child  link="diana_gripper/left_finger_proximal_servo" />
+  <xacro:scservo name="${name}/left_finger_proximal_servo"
+                 type="scs20"
+                 rgba="0.0 0.0 0.6 1.0" gmaterial="Gazebo/Blue">
+  </xacro:scservo>
+  <xacro:scservo name="${name}/left_finger_distal_servo"
+                 type="scs20"
+                 rgba="0.0 0.0 0.6 1.0" gmaterial="Gazebo/Blue">
+  </xacro:scservo>
+  <xacro:scservo name="${name}/right_finger_proximal_servo"
+                 type="scs20"
+                 rgba="0.0 0.0 0.6 1.0" gmaterial="Gazebo/Blue">
+  </xacro:scservo>
+  <xacro:scservo name="${name}/right_finger_distal_servo"
+                 type="scs20"
+                 rgba="0.0 0.0 0.6 1.0" gmaterial="Gazebo/Blue">
+  </xacro:scservo>
+  <joint name="${name}/left_finger_proximal_servo_mount_joint" type="fixed" >
+    <parent link="${name}" />
+    <child  link="${name}/left_finger_proximal_servo" />
     <origin xyz="${-0.075+0.01} 0 ${0.015+0.005+0.03}" rpy="0 3.1415 0" />
   </joint>
-  <joint name="diana_gripper/LFJ2" type="revolute" >
-    <parent link="diana_gripper/left_finger_proximal_servo" />
-    <child  link="diana_gripper/left_finger_connector" />
+  <joint name="${name}/LFJ2" type="revolute" >
+    <parent link="${name}/left_finger_proximal_servo" />
+    <child  link="${name}/left_finger_connector" />
     <origin xyz="0 0 0" rpy="0 0 0" />
     <axis xyz="0 1 0" />
@@ -77,18 +77,18 @@
     <safety_controller soft_lower_limit="-1.57" soft_upper_limit="1.57" k_position="1000" k_velocity="100"/>
   </joint>
-  <transmission name="diana_gripper/LFJ2_joint_transmission">
-    <type>transmission_interface/SimpleTransmission</type>
-    <joint name="diana_gripper/LFJ2" >
-      <hardwareInterface>hardware_interface/EffortJointInterface</hardwareInterface>
-    </joint>
-    <actuator name="diana_gripper/left_finger_proximal_joint_motor" >
-      <hardwareInterface>hardware_interface/EffortJointInterface</hardwareInterface>
-      <mechanicalReduction>100</mechanicalReduction>
-    </actuator>
-  </transmission>
-  <link name="diana_gripper/left_finger_connector" >
-    <visual>
-      <origin xyz="0 0.001 0" rpy="0 -1.571 0" />
-      <material name="diana_gripper_left_finger_connector_material" >
+  <transmission name="${name}/LFJ2_joint_transmission">
+    <type>transmission_interface/SimpleTransmission</type>
+    <joint name="${name}/LFJ2" >
+      <hardwareInterface>hardware_interface/EffortJointInterface</hardwareInterface>
+    </joint>
+    <actuator name="${name}/left_finger_proximal_joint_motor" >
+      <hardwareInterface>hardware_interface/EffortJointInterface</hardwareInterface>
+      <mechanicalReduction>100</mechanicalReduction>
+    </actuator>
+  </transmission>
+  <link name="${name}/left_finger_connector" >
+    <visual>
+      <origin xyz="0 0.001 0" rpy="0 -1.571 0" />
+      <material name="${name}_left_finger_connector_material" >
         <color rgba="1.0 0.0 0.0 1.0" />
       </material>
@@ -104,13 +104,13 @@
     </collision>
   </link>
-  <joint name="diana_gripper/left_finger_distal_servo_mount_joint" type="fixed" >
-    <parent link="diana_gripper/left_finger_connector" />
-    <child  link="diana_gripper/left_finger_distal_servo" />
+  <joint name="${name}/left_finger_distal_servo_mount_joint" type="fixed" >
+    <parent link="${name}/left_finger_connector" />
+    <child  link="${name}/left_finger_distal_servo" />
     <origin xyz="0 0 ${-0.03-0.017}" rpy="0 0 0" />
   </joint>
-  <link name="diana_gripper/left_finger_distal_bracket" >
-    <visual>
-      <origin xyz="0 0 -0.0275" rpy="0 0 1.571" />
-      <material name="diana_gripper_left_finger_distal_bracket_material" >
+  <link name="${name}/left_finger_distal_bracket" >
+    <visual>
+      <origin xyz="0 0 -0.0275" rpy="0 0 1.571" />
+      <material name="${name}_left_finger_distal_bracket_material" >
         <color rgba="0.9 0.9 0.9 1.0" />
       </material>
@@ -126,7 +126,7 @@
     </collision>
   </link>
-  <joint name="diana_gripper/LFJ1" type="revolute" >
-    <parent link="diana_gripper/left_finger_distal_servo" />
-    <child  link="diana_gripper/left_finger_distal_bracket" />
+  <joint name="${name}/LFJ1" type="revolute" >
+    <parent link="${name}/left_finger_distal_servo" />
+    <child  link="${name}/left_finger_distal_bracket" />
     <origin xyz="0 0 0" rpy="0 0 0" />
     <axis xyz="0 1 0" />
@@ -135,30 +135,30 @@
     <safety_controller soft_lower_limit="-2.20" soft_upper_limit="2.20" k_position="1000" k_velocity="100"/>
   </joint>
-  <transmission name="diana_gripper/LFJ1_joint_transmission">
-    <type>transmission_interface/SimpleTransmission</type>
-    <joint name="diana_gripper/LFJ1" >
-      <hardwareInterface>hardware_interface/EffortJointInterface</hardwareInterface>
-    </joint>
-    <actuator name="diana_gripper/left_finger_distal_joint_motor" >
-      <hardwareInterface>hardware_interface/EffortJointInterface</hardwareInterface>
-      <mechanicalReduction>100</mechanicalReduction>
-    </actuator>
-  </transmission>
-  <link name="diana_gripper/left_finger_tip_mount" />
+  <transmission name="${name}/LFJ1_joint_transmission">
+    <type>transmission_interface/SimpleTransmission</type>
+    <joint name="${name}/LFJ1" >
+      <hardwareInterface>hardware_interface/EffortJointInterface</hardwareInterface>
+    </joint>
+    <actuator name="${name}/left_finger_distal_joint_motor" >
+      <hardwareInterface>hardware_interface/EffortJointInterface</hardwareInterface>
+      <mechanicalReduction>100</mechanicalReduction>
+    </actuator>
+  </transmission>
+  <link name="${name}/left_finger_tip_mount" />
   <!-- convert from weird SCS20 coordinates back to base frame (when finger straight) -->
-  <joint name="diana_gripper/left_finger_tip_mount_joint" type="fixed">
-    <parent link="diana_gripper/left_finger_distal_bracket" />
-    <child  link="diana_gripper/left_finger_tip_mount" />
+  <joint name="${name}/left_finger_tip_mount_joint" type="fixed">
+    <parent link="${name}/left_finger_distal_bracket" />
+    <child  link="${name}/left_finger_tip_mount" />
     <origin xyz="0 0 ${-0.0275}" rpy="0 3.1415 0" />
   </joint>
   <!-- right finger with joints -->
-  <joint name="diana_gripper/right_finger_proximal_servo_mount_joint" type="fixed" >
-    <parent link="diana_gripper" />
-    <child  link="diana_gripper/right_finger_proximal_servo" />
+  <joint name="${name}/right_finger_proximal_servo_mount_joint" type="fixed" >
+    <parent link="${name}" />
+    <child  link="${name}/right_finger_proximal_servo" />
     <origin xyz="${+0.075-0.01} 0 ${0.015+0.005+0.03}" rpy="0 3.1415 0" />
   </joint>
-  <joint name="diana_gripper/RFJ2" type="revolute" >
-    <parent link="diana_gripper/right_finger_proximal_servo" />
-    <child  link="diana_gripper/right_finger_connector" />
+  <joint name="${name}/RFJ2" type="revolute" >
+    <parent link="${name}/right_finger_proximal_servo" />
+    <child  link="${name}/right_finger_connector" />
     <origin xyz="0 0 0" rpy="0 0 0" />
     <axis xyz="0 -1 0" />
@@ -167,18 +167,18 @@
     <safety_controller soft_lower_limit="-1.57" soft_upper_limit="1.57" k_position="1000" k_velocity="100"/>
   </joint>
-  <transmission name="diana_gripper/RFJ2_joint_transmission">
-    <type>transmission_interface/SimpleTransmission</type>
-    <joint name="diana_gripper/RFJ2" >
-      <hardwareInterface>hardware_interface/EffortJointInterface</hardwareInterface>
-    </joint>
-    <actuator name="diana_gripper/RFJ2_joint_motor" >
-      <hardwareInterface>hardware_interface/EffortJointInterface</hardwareInterface>
-      <mechanicalReduction>100</mechanicalReduction>
-    </actuator>
-  </transmission>
-  <link name="diana_gripper/right_finger_connector" >
-    <visual>
-      <origin xyz="0 0.001 0" rpy="0 -1.571 0" />
-      <material name="diana_gripper_right_finger_connector_material" >
+  <transmission name="${name}/RFJ2_joint_transmission">
+    <type>transmission_interface/SimpleTransmission</type>
+    <joint name="${name}/RFJ2" >
+      <hardwareInterface>hardware_interface/EffortJointInterface</hardwareInterface>
+    </joint>
+    <actuator name="${name}/RFJ2_joint_motor" >
+      <hardwareInterface>hardware_interface/EffortJointInterface</hardwareInterface>
+      <mechanicalReduction>100</mechanicalReduction>
+    </actuator>
+  </transmission>
+  <link name="${name}/right_finger_connector" >
+    <visual>
+      <origin xyz="0 0.001 0" rpy="0 -1.571 0" />
+      <material name="${name}_right_finger_connector_material" >
         <color rgba="0.0 1.0 0.0 1.0" />
       </material>
@@ -194,13 +194,13 @@
     </collision>
   </link>
-  <joint name="diana_gripper/right_finger_distal_servo_mount_joint" type="fixed" >
-    <parent link="diana_gripper/right_finger_connector" />
-    <child  link="diana_gripper/right_finger_distal_servo" />
+  <joint name="${name}/right_finger_distal_servo_mount_joint" type="fixed" >
+    <parent link="${name}/right_finger_connector" />
+    <child  link="${name}/right_finger_distal_servo" />
     <origin xyz="0 0 ${-0.03-0.017}" rpy="0 0 0" />
   </joint>
-  <link name="diana_gripper/right_finger_distal_bracket" >
-    <visual>
-      <origin xyz="0 0 -0.0275" rpy="0 0 1.571" />
-      <material name="diana_gripper_right_finger_distal_bracket_material" >
+  <link name="${name}/right_finger_distal_bracket" >
+    <visual>
+      <origin xyz="0 0 -0.0275" rpy="0 0 1.571" />
+      <material name="${name}_right_finger_distal_bracket_material" >
         <color rgba="0.9 0.9 0.9 1.0" />
       </material>
@@ -216,7 +216,7 @@
     </collision>
   </link>
-  <joint name="diana_gripper/RFJ1" type="revolute" >
-    <parent link="diana_gripper/right_finger_distal_servo" />
-    <child  link="diana_gripper/right_finger_distal_bracket" />
+  <joint name="${name}/RFJ1" type="revolute" >
+    <parent link="${name}/right_finger_distal_servo" />
+    <child  link="${name}/right_finger_distal_bracket" />
     <origin xyz="0 0 0" rpy="0 0 0" />
     <axis xyz="0 -1 0" />
@@ -225,19 +225,19 @@
     <safety_controller soft_lower_limit="-2.20" soft_upper_limit="2.20" k_position="1000" k_velocity="100"/>
   </joint>
-  <transmission name="diana_gripper/RFJ1_joint_transmission">
-    <type>transmission_interface/SimpleTransmission</type>
-    <joint name="diana_gripper/RFJ1" >
-      <hardwareInterface>hardware_interface/EffortJointInterface</hardwareInterface>
-    </joint>
-    <actuator name="diana_gripper/RFJ1_joint_motor" >
-      <hardwareInterface>hardware_interface/EffortJointInterface</hardwareInterface>
-      <mechanicalReduction>100</mechanicalReduction>
-    </actuator>
-  </transmission>
-  <link name="diana_gripper/right_finger_tip_mount" />
+  <transmission name="${name}/RFJ1_joint_transmission">
+    <type>transmission_interface/SimpleTransmission</type>
+    <joint name="${name}/RFJ1" >
+      <hardwareInterface>hardware_interface/EffortJointInterface</hardwareInterface>
+    </joint>
+    <actuator name="${name}/RFJ1_joint_motor" >
+      <hardwareInterface>hardware_interface/EffortJointInterface</hardwareInterface>
+      <mechanicalReduction>100</mechanicalReduction>
+    </actuator>
+  </transmission>
+  <link name="${name}/right_finger_tip_mount" />
   <!-- convert from weird SCS20 coordinates back to base frame (when finger straight) -->
-  <joint name="diana_gripper/right_finger_tip_mount_joint" type="fixed">
-    <parent link="diana_gripper/right_finger_distal_bracket" />
-    <child  link="diana_gripper/right_finger_tip_mount" />
+  <joint name="${name}/right_finger_tip_mount_joint" type="fixed">
+    <parent link="${name}/right_finger_distal_bracket" />
+    <child  link="${name}/right_finger_tip_mount" />
     <origin xyz="0 0 ${-0.0275}" rpy="0 3.1415 0" />   <!-- or ${-0.0275-0.02} -->
   </joint>
@@ -248,8 +248,8 @@
   <xacro:simple_fingertips/>  -->
   <xacro:tcp/>
-  <xacro:imu_gy521 parent="diana_gripper/left_finger_tip_mount" name="diana_gripper/left_finger_imu" >
+  <xacro:imu_gy521 parent="${name}/left_finger_tip_mount" name="${name}/left_finger_imu" >
     <origin xyz="0 0.023 0" rpy="0 0 3.141" />
   </xacro:imu_gy521>
-  <xacro:imu_gy521 parent="diana_gripper/right_finger_tip_mount" name="diana_gripper/right_finger_imu" >
+  <xacro:imu_gy521 parent="${name}/right_finger_tip_mount" name="${name}/right_finger_imu" >
     <origin xyz="0 0.023 0" rpy="0 0 3.141" />
   </xacro:imu_gy521>

Commit message: added usb hub to base collision object

File: urdf/diana_gripper.xacro (robot description, xacro)
@@ -30,7 +30,7 @@
       <!-- one single lump as a collision block, covers base plate, four load cells, two servo carriers -->
       <collision>
-        <origin xyz="0 0 ${(0.02+0.0127)/2}" rpy="0 0 0" />
+        <origin xyz="0 0.025 ${(0.02+0.0127)/2}" rpy="0 0 0" />
         <geometry>
-          <box size="${0.075*2} 0.105 ${0.02+0.0127}" />
+          <box size="${0.075*2} ${0.105 + 0.05} ${0.02+0.0127}" />
         </geometry>
       </collision>

Commit message: Add missing inertial blocks.

File: urdf/diana_gripper.xacro (robot description, xacro)
@@ -6,5 +6,5 @@
   <xacro:include filename="$(find diana_gripper)/urdf/imu_gy521.xacro" />
   <xacro:include filename="$(find diana_gripper)/urdf/fingertip.xacro" />
-  <xacro:diana_gripper_control_plugin name="diana_gripper" />
+  <!-- <xacro:diana_gripper_control_plugin name="diana_gripper" /> -->
 <xacro:macro name="diana_gripper" params="name" >
   <!-- prototype two-finger diana_gripper with four SC servos.
@@ -88,4 +88,9 @@
   </transmission>
   <link name="${name}/left_finger_connector" >
+    <inertial>
+      <origin xyz="0 0 0" rpy="0 0 0"/>
+      <mass value="0.011" />
+      <inertia ixx="0.001" ixy="0" ixz="0" iyy="0.001" iyz="0" izz="0.001" />
+    </inertial>
     <visual>
       <origin xyz="0 0.001 0" rpy="0 -1.571 0" />
@@ -110,4 +115,9 @@
   </joint>
   <link name="${name}/left_finger_distal_bracket" >
+    <inertial>
+      <origin xyz="0 0 0" rpy="0 0 0"/>
+      <mass value="0.011" />
+      <inertia ixx="0.001" ixy="0" ixz="0" iyy="0.001" iyz="0" izz="0.001" />
+    </inertial>
     <visual>
       <origin xyz="0 0 -0.0275" rpy="0 0 1.571" />
@@ -178,4 +188,9 @@
   </transmission>
   <link name="${name}/right_finger_connector" >
+    <inertial>
+      <origin xyz="0 0 0" rpy="0 0 0"/>
+      <mass value="0.011" />
+      <inertia ixx="0.001" ixy="0" ixz="0" iyy="0.001" iyz="0" izz="0.001" />
+    </inertial>
     <visual>
       <origin xyz="0 0.001 0" rpy="0 -1.571 0" />
@@ -200,4 +215,9 @@
   </joint>
   <link name="${name}/right_finger_distal_bracket" >
+    <inertial>
+      <origin xyz="0 0 0" rpy="0 0 0"/>
+      <mass value="0.011" />
+      <inertia ixx="0.001" ixy="0" ixz="0" iyy="0.001" iyz="0" izz="0.001" />
+    </inertial>
     <visual>
       <origin xyz="0 0 -0.0275" rpy="0 0 1.571" />
@@ -247,4 +267,8 @@
   <xacro:finray_ridges_fingertips/>
   <xacro:simple_fingertips/>  -->
+<!--
+  diana_gripper/left_fingertip
+  diana_gripper/right_fingertip
+-->
   <xacro:tcp/>
   <xacro:imu_gy521 parent="${name}/left_finger_tip_mount" name="${name}/left_finger_imu" >

Commit message: merge xacro

File: urdf/diana_gripper.xacro (robot description, xacro)
@@ -271,5 +271,5 @@
   diana_gripper/right_fingertip
 -->
-  <xacro:tcp/>
+  <xacro:tcp name="${name}"/>
   <xacro:imu_gy521 parent="${name}/left_finger_tip_mount" name="${name}/left_finger_imu" >
     <origin xyz="0 0.023 0" rpy="0 0 3.141" />
@@ -295,10 +295,10 @@
   </joint>
 </xacro:macro>
-<xacro:macro name="tcp">
-  <link name="diana_gripper/tcp" >
-  </link>
-  <joint name="diana_gripper/tcp_joint" type="fixed" >
-    <parent link="diana_gripper" />
-    <child  link="diana_gripper/tcp" />
+<xacro:macro name="tcp" params="name">
+  <link name="${name}/tcp" >
+  </link>
+  <joint name="${name}/tcp_joint" type="fixed" >
+    <parent link="${name}" />
+    <child  link="${name}/tcp" />
     <origin xyz="0 0 0.15" rpy="0 0 0" />
   </joint>
